File: hardware/devboard/board/Yapogee-Devboard/MCU.kicad_sch (KiCad schematic)
At the start: 1 part, among them U1 RP2350B_SC1510_A4

Commit message: AAAAAAAAAA
Parts:
- added C1, C34, C35, C36, C37, C38, C39, C40, C41, C42, C43, C44, C45, C48, C52: 100nF, Yapogee:C_Murata_GCM15_1005_RefReflow, symbol Yapogee:GCM155R71H104KE02D
- added C31, C32, C46, C49: 4.7uF, Yapogee:C_Murata_GRM15_RP2350_Core_Ref, symbol Yapogee:GRM155R60J475ME47D
- added C47: 22uF, Yapogee:C_Murata_GCM31_3216_RefReflow, symbol Yapogee:GCM31CR71A226KE02L
- added L3: 3.3uH, Yapogee:Abracon_AOTA_B201610S3R3_101_T, symbol Yapogee:AOTA_B201610S3R3_101_T
- added R33, R34: 27Ω, Yapogee:R_0402_1005Metric, symbol Yapogee:0402,27Ω
- added R35, R36: 1kΩ, Yapogee:R_0402_1005Metric, symbol Yapogee:0402,1kΩ
- added R37: 33Ω, Yapogee:R_0402_1005Metric, symbol Yapogee:0402,33Ω
- added R40: 0Ω, Yapogee:R_0402_1005Metric, symbol Yapogee:0402,0Ω
- added SW1, SW2: EVPBB2A9B000, Yapogee:Panasonic_EVPBB_2.6x1.6mm, symbol Yapogee:EVPBB2A9B000
- added TP13: SWCLK, TestPoint:TestPoint_Pad_D1.5mm, symbol Yapogee:TestPoint_Pad_1mm
- added TP14: SWDIO, TestPoint:TestPoint_Pad_D1.5mm, symbol Yapogee:TestPoint_Pad_1mm
- added TP15: GND, TestPoint:TestPoint_Pad_D1.5mm, symbol Yapogee:TestPoint_Pad_1mm
- added U16: SN74LVC1G125DBVR, Yapogee:SN74LVC1G125DBVR, symbol Yapogee:SN74LVC1G125DBVR
- added U3: W25Q128JVSIQ, Yapogee:SOIC-8_5.3x5.3mm_P1.27mm, symbol Yapogee:W25Q128JVSIQ
- U2: renamed from U1; Device (none) -> RP2350B0A4; MPN (none) -> SC1510-A4; Manufacturer (none) -> Raspberry Pi; Stepping (none) -> A4
Connections:
- net CORE_1V1: now reaches U2.10 (DVDD)
- net CORE_1V1: now also U2.32 (DVDD), U2.51 (DVDD), U2.65 (VREG_FB), C43.1, C44.1, C45.1, C46.1, C49.1, L3.1
- net DIG_3V3: now reaches U2.15 (IOVDD)
- net DIG_3V3: now also U2.24 (IOVDD), U2.29 (IOVDD), U2.41 (IOVDD), U2.5 (IOVDD), U2.50 (IOVDD), U2.59 (ADC_AVDD), U2.60 (IOVDD), U2.64 (VREG_VIN), U2.68 (USB_OTP_VDD), U2.69 (QSPI_IOVDD), U2.76 (IOVDD), C1.1, C31.1, C34.1, C35.1, C36.1, C37.1, C38.1, C39.1, C40.1, C41.1, C42.1, C47.1, C48.1, C52.2, R37.1, U16.5 (VCC), U3.8 (VCC)
- net at U2.61 (VREG_AVDD): now also C32.1, R37.2
- net GND: now reaches U2.62 (VREG_PGND)
- net GND: now also U2.81 (GND), C1.2, C31.2, C32.2, C34.2, C35.2, C36.2, C37.2, C38.2, C39.2, C40.2, C41.2, C42.2, C43.2, C44.2, C45.2, C46.2, C47.2, C48.2, C49.2, C52.1, SW1.2, SW2.2, TP15.1, U16.1 (~{OE}), U16.3 (GND), U3.4 (GND)
- net at U2.63 (VREG_LX): now also L3.2
- net at U2.30 (XIN): now also R40.2
- net SWCLK: now reaches U2.33 (SWCLK)
- net SWCLK: now also TP13.1
- net SWDIO: now reaches U2.34 (SWDIO)
- net SWDIO: now also TP14.1
- net RUN_N: now reaches U2.35 (RUN)
- net RUN_N: now also R36.1
- net at U2.66 (USB_DM): now also R33.1
- net at U2.67 (USB_DP): now also R34.1
- net at U2.70 (QSPI_SD3): now also U3.7 (IO3_/_~{HOLD})
- net at U2.71 (QSPI_SCLK): now also U3.6 (CLK)
- net at U2.72 (QSPI_SD0): now also U3.5 (IO0_/_DI)
- net at U2.73 (QSPI_SD2): now also U3.3 (IO2_/_~{WP})
- net at U2.74 (QSPI_SD1): now also U3.2 (IO1_/_DO)
- net QSPI_CS_N: now reaches U2.75 (~{QSPI_SS})
- net QSPI_CS_N: now also R35.1, U3.1 (~{CS})
- new net: R40.1, U16.4 (Y)
- new net: R36.2, SW2.1
- new net: R35.2, SW1.1
- new net REF_12M: U16.2 (A)
- new net USB_N: R33.2
- new net USB_P: R34.2
- no-connect marks 0 -> 1
Other:
- note added: "10 / 32 / 51; 4.7 µF near 32"
- note added: "ADC"
- note added: "BOOTSEL"
- note added: "Boot"
- note added: "DVDD"
- note added: "Decoupling"
- note added: "General GPIO"
- note added: "IOVDD"
- note added: "MCU Power"
- note added: "MCU Timing and QSPI"
- note added: "Near pins 5 / 15 / 24 / 29 / 41 / 50 / 60 / 76"
- note added: "Pin 59"
- note added: "RP2350B"
- note added: "RST"
- note added: "RUN"
- note added: "SWD"
- note added: "Waveform GPIO"
- company: (none) -> Yapogee
- title: (none) -> MCU
- moved on the sheet: U2A, U2B, U2D
