File: hardware/devboard/board/Yapogee-Devboard/Yapogee-Devboard.kicad_sch (KiCad schematic)
At the start: 0 parts

Commit message: yuh yuh
Other:
- added sheet MCU (MCU.kicad_sch)
- note added: "A Rivercraft Creation"
- note added: "I/Q generation and control"
- note added: "Something witty about yapping from apogee"
- note added: "Yapogee Devboard"
Changed lines of the file:
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@@
 	(generator_version "10.0")
 	(paper "A4")
+	(text "Yapogee Devboard"
+		(exclude_from_sim no)
+		(at 144.272 26.67 0)
+		(effects
+			(font
+				(face "Trebuchet MS")
+				(size 7 7)
+				(thickness 1.4)
+				(bold yes)
+			)
+		)
+	)
+	(text "Something witty about yapping from apogee\n"
+		(exclude_from_sim no)
+		(at 145.542 34.036 0)
+		(effects
+			(font
+				(face "Trebuchet MS")
+				(size 3 3)
+				(thickness 1.4)
+				(bold yes)
+			)
+		)
+	)
+	(text "I/Q generation and control"
+		(exclude_from_sim no)
+		(at 115.316 90.932 0)
+		(effects
+			(font
+				(size 2 2)
+				(thickness 0.4)
+				(bold yes)
+			)
+		)
+	)
+	(text "A Rivercraft Creation\n\n"
+		(exclude_from_sim no)
+		(at 145.542 42.418 0)
+		(effects
+			(font
+				(face "Trebuchet MS")
+				(size 3 3)
+				(thickness 1.4)
+				(bold yes)
+			)
+		)
+	)
+	(sheet
+		(at 85.725 86.995)
+		(size 60.96 50.8)
+		(exclude_from_sim no)
+		(in_bom yes)
+		(on_board yes)
+		(dnp no)
+		(stroke
+			(width 0.1524)
+			(type solid)
+		)
+		(fill
+			(color 0 0 0 0)
+		)
+		(property "Sheetname" "MCU"
+			(at 109.982 86.614 0)
+			(show_name no)
+			(do_not_autoplace no)
+			(effects
+				(font
+					(size 3 3)
+					(thickness 1)
+					(bold yes)
+				)
+				(justify left bottom)
+			)
+		)
+		(property "Sheetfile" "MCU.kicad_sch"
+			(at 85.725 138.3796 0)
+			(show_name no)
+			(do_not_autoplace no)
+			(effects
+				(font
+					(size 1.27 1.27)
+				)
+				(justify left top)
+			)
+		)
+		(instances
+			(project "Yapogee-Devboard"
+				(path "/111c3c71-9370-42b8-a37f-1eaf0b24b42b"
+					(page "2")
+				)
+			)
+		)
+	)
 	(sheet_instances
 		(path "/"

Commit message: AAAAAAAAAA
Parts:
- added J1: Conn_01x02, symbol Connector_Generic:Conn_01x02
- added J2: USB4105-GF-A, Yapogee:USB4105-GF-A, symbol Yapogee:USB4105-GF-A
- added JP1: USB_PWR_LINK, Yapogee:SolderJumper-2_P1.3mm_Open_Pad1.0x1.5mm, symbol Yapogee:SolderJumper_2_Bridged
- added R1, R2: 5.1kΩ, PCM_JLCPCB:R_0402, symbol PCM_JLCPCB-Resistors:0402,5.1kΩ
- added U1: TPD2EUSB30DRTR, Yapogee:TPD2EUSB30DRTR, symbol Yapogee:TPD2EUSB30DRTR
Connections:
- new net: J2.A4 (VBUS), J2.A9 (VBUS), J2.B4 (VBUS), J2.B9 (VBUS), JP1.1 (A)
- new net: J2.A5 (CC1), R1.1
- new net: J2.B5 (CC2), R2.1
- new net GND: J1.1 (Pin_1), J2.A1 (GND), J2.A12 (GND), J2.B1 (GND), J2.B12 (GND), J2.SH (SHIELD), R1.2, R2.2, U1.3 (GND)
- new net Power/5V_IN: J1.2 (Pin_2), JP1.2 (B)
- new net USB_N: J2.A7 (D-), J2.B7 (D-), U1.2 (D-)
- new net USB_P: J2.A6 (D+), J2.B6 (D+), U1.1 (D+)
- no-connect marks 0 -> 2
Other:
- added sheet IQ & RF Front End (IQ_RF_FRONT_END.kicad_sch)
- added sheet LO & 12 MHz Clock Fanout (LO_Clocks.kicad_sch)
- added sheet Power (Power.kicad_sch)
- sheet MCU ports: added REF_12M, USB_N, USB_P; removed none
- note added: "12.5 MHz to 6.4 GHz LO"
- note added: "12MHz TCXO Fanout"
- note added: "5V In"
- note added: "5V, 3V3, 2V5, 1V8"
- note added: "Bridge when only using USB power"
- note added: "Insert something witty about yapping from apogee"
- note removed: "Something witty about yapping from apogee"
